Commit message: changed robot class to be reconfigurable

File: aerial_gym_ws/src/aerial_gym_simulator/resources/robots/flapper/flapper_simple.urdf (robot description, URDF)
Before this commit: robot flapper, 5 links, 4 joints
Joints:
- joint left_wing_back_m: axis 0.0 -1.0 0.0 -> 0.0 0.0 -1.0; limit lower=-0.785398 upper=0.0 effort=100 velocity=100 -> (none); type fixed -> revolute
- joint left_wing_front: axis 0.0 -1.0 0.0 -> 0.0 0.0 1.0; limit lower=0.0 upper=0.785398 effort=100 velocity=100 -> (none); type fixed -> revolute
- joint right_wing_back: axis 0.0 -1.0 0.0 -> 0.0 0.0 -1.0; limit lower=0.0 upper=0.785398 effort=100 velocity=100 -> (none); type fixed -> revolute
- joint right_wing_front_m: axis 0.0 -1.0 0.0 -> 0.0 0.0 1.0; limit lower=-0.785398 upper=0.0 effort=100 velocity=100 -> (none); type fixed -> revolute
